File: boards/chromatone/chromatone.kicad_sch (KiCad schematic)
At the start: 0 parts

Commit message: chromatone: schematic (ISO7720 isolated SPI, both domains, ERC clean)
Co-Authored-By: Claude Fable 5.1 <noreply@anthropic.com>
Parts:
- added C1, C3: 100n, Capacitor_SMD:C_0603_1608Metric, symbol Device:C
- added C2, C4: 10u, Capacitor_SMD:C_0603_1608Metric, symbol Device:C
- added D1: GREEN, LED_SMD:LED_0603_1608Metric, symbol Device:LED
- added D2: BLUE, LED_SMD:LED_0603_1608Metric, symbol Device:LED
- added H1, H2, H3, H4: M2.5, MountingHole:MountingHole_2.7mm_M2.5, symbol Mechanical:MountingHole
- added J1: Pi SPI, Connector_JST:JST_XH_B4B-XH-A_1x04_P2.50mm_Vertical, symbol Connector:Conn_01x04_Pin
- added J2: Strip, Connector_JST:JST_XH_B4B-XH-A_1x04_P2.50mm_Vertical, symbol Connector:Conn_01x04_Pin
- added R1, R2: 47, Resistor_SMD:R_0603_1608Metric, symbol Device:R
- added R3, R4: 1k, Resistor_SMD:R_0603_1608Metric, symbol Device:R
- added TP1: SCLK, TestPoint:TestPoint_Pad_D1.5mm, symbol Connector:TestPoint
- added TP2: MOSI, TestPoint:TestPoint_Pad_D1.5mm, symbol Connector:TestPoint
- added TP3: CLK, TestPoint:TestPoint_Pad_D1.5mm, symbol Connector:TestPoint
- added TP4: DATA, TestPoint:TestPoint_Pad_D1.5mm, symbol Connector:TestPoint
- added U1: ISO7720D, Package_SO:SOIC-8_3.9x4.9mm_P1.27mm, symbol Isolator:ISO7720D
Connections:
- new net: J1.2 (Pin_2), TP1.1, U1.2 (INA)
- new net: J1.3 (Pin_3), TP2.1, U1.3 (INB)
- new net: R2.1, U1.6 (OUTB)
- new net: R1.1, U1.7 (OUTA)
- new net: D1.2 (A), R3.2
- new net: J2.2 (Pin_2), R1.2, TP3.1
- new net: J2.3 (Pin_3), R2.2, TP4.1
- new net: D2.2 (A), R4.2
- new net +3V3: C1.1, C2.1, J1.1 (Pin_1), R3.1, U1.1 (VCC1)
- new net +5V_LED: C3.1, C4.1, J2.1 (Pin_1), R4.1, U1.8 (VCC2)
- new net GND: C1.2, C2.2, D1.1 (K), J1.4 (Pin_4), U1.4 (GND1)
- new net GND_LED: C3.2, C4.2, D2.1 (K), J2.4 (Pin_4), U1.5 (GND2)
Other:
- note added: "DOMAIN A: Pi side, 3.3 V, Pi battery"
- note added: "DOMAIN B: LED side, 5 V, LED battery"
- note added: "Isolation barrier: only SPI CLK and DATA cross, A -> B. GND and GND_LED never touch."
- note added: "J1 to Pi header: 1=3V3 (pin 1), 2=SCLK (GPIO11), 3=MOSI (GPIO10), 4=GND."
- note added: "J2 to pixel 0 of the strip: 1=5V, 2=CI, 3=DI, 4=GND. Tap 5V/GND at the strip end so VCC2 never exceeds the pixel rail."
- note added: "R1/R2 tame ringing on the CLK/DATA leads; keep leads to pixel 0 short, twisted with GND_LED."
- title: chromatone -> Chromatone isolated SPI daughterboard

Commit message: chromatone: PCB layout rev A (46x30 mm, split ground pours, 3 mm barrier) + generators
DRC clean with warnings and schematic parity; make jlcpcb runs end to end.

Co-Authored-By: Claude Fable 5.1 <noreply@anthropic.com>
Parts:
- H1, H2, H3, H4, TP1, TP2, TP3, TP4: now left out of the parts list
Changed lines of the file:
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@@
 		(unit 1)
 		(exclude_from_sim no)
-		(in_bom yes)
+		(in_bom no)
 		(on_board yes)
 		(dnp no)
@@
 		(unit 1)
 		(exclude_from_sim no)
-		(in_bom yes)
+		(in_bom no)
 		(on_board yes)
 		(dnp no)
@@
 		(unit 1)
 		(exclude_from_sim no)
-		(in_bom yes)
+		(in_bom no)
 		(on_board yes)
 		(dnp no)
@@
 		(unit 1)
 		(exclude_from_sim no)
-		(in_bom yes)
+		(in_bom no)
 		(on_board yes)
 		(dnp no)
@@
 		(unit 1)
 		(exclude_from_sim no)
-		(in_bom yes)
+		(in_bom no)
 		(on_board yes)
 		(dnp no)
@@
 		(unit 1)
 		(exclude_from_sim no)
-		(in_bom yes)
+		(in_bom no)
 		(on_board yes)
 		(dnp no)
@@
 		(unit 1)
 		(exclude_from_sim no)
-		(in_bom yes)
+		(in_bom no)
 		(on_board yes)
 		(dnp no)
@@
 		(unit 1)
 		(exclude_from_sim no)
-		(in_bom yes)
+		(in_bom no)
 		(on_board yes)
 		(dnp no)

Commit message: chromatone: review fixes (JST LCSC C144395, decoupling at U1 pins, hole keepouts, ground test pads, 8 MHz target)
Co-Authored-By: Claude Fable 5.1 <noreply@anthropic.com>
Parts:
- added TP5: GND_A, TestPoint:TestPoint_Pad_D1.5mm, symbol Connector:TestPoint
- added TP6: GND_B, TestPoint:TestPoint_Pad_D1.5mm, symbol Connector:TestPoint
- J1, J2: LCSC C144394 -> C144395
Connections:
- net GND: now also TP5.1
- net GND_LED: now also TP6.1
Changed lines of the file:
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@@
 			)
 		)
-		(property "LCSC" "C144394"
+		(property "LCSC" "C144395"
 			(at 58.42 48.26 0)
 			(effects
@@
 			)
 		)
-		(property "LCSC" "C144394"
+		(property "LCSC" "C144395"
 			(at 148.59 48.26 0)
 			(effects
@@
 			)
 		)
-		(property "Description" "Unpolarized capacitor"
+		(property "Description" "100 nF X7R 50 V"
 			(at 74.93 69.85 0)
 			(effects
@@
 			)
 		)
-		(property "Description" "Unpolarized capacitor"
+		(property "Description" "10 uF X5R 10 V"
 			(at 85.09 69.85 0)
 			(effects
@@
 		)
 	)
+	(junction
+		(at 68.58 76.2)
+		(diameter 0)
+		(color 0 0 0 0)
+	)
+	(symbol
+		(lib_id "Connector:TestPoint")
+		(at 68.58 76.2 180)
+		(unit 1)
+		(exclude_from_sim no)
+		(in_bom no)
+		(on_board yes)
+		(dnp no)
+		(property "Reference" "TP5"
+			(at 66.58 82.9 0)
+			(effects
+				(font
+					(size 1.27 1.27)
+				)
+			)
+		)
+		(property "Value" "GND_A"
+			(at 66.58 81 0)
+			(effects
+				(font
+					(size 1.27 1.27)
+				)
+			)
+		)
+		(property "Footprint" "TestPoint:TestPoint_Pad_D1.5mm"
+			(at 71.12 76.2 0)
+			(effects
+				(font
+					(size 1.27 1.27)
+				)
+				(hide yes)
+			)
+		)
+		(property "Datasheet" ""
+			(at 71.12 76.2 0)
+			(effects
+				(font
+					(size 1.27 1.27)
+				)
+				(hide yes)
+			)
+		)
+		(property "Description" "test point"
+			(at 71.12 76.2 0)
+			(effects
+				(font
+					(size 1.27 1.27)
+				)
+				(hide yes)
+			)
+		)
+		(pin "1"
+		)
+		(instances
+			(project "chromatone"
+				(path "/25fa9059-b474-40ad-8d4e-edcbfb8482a5"
+					(reference "TP5")
+					(unit 1)
+				)
+			)
+		)
+	)
 	(symbol
 		(lib_id "Device:R")
@@
 			)
 		)
-		(property "Description" "Unpolarized capacitor"
+		(property "Description" "100 nF X7R 50 V"
 			(at 124.46 69.85 0)
 			(effects
@@
 			)
 		)
-		(property "Description" "Unpolarized capacitor"
+		(property "Description" "10 uF X5R 10 V"
 			(at 134.62 69.85 0)
 			(effects
@@
 					(unit 1)
 				)
+			)
+		)
+	)
+	(junction
+		(at 118.11 76.2)
+		(diameter 0)
+		(color 0 0 0 0)
+	)
+	(symbol
+		(lib_id "Connector:TestPoint")
+		(at 118.11 76.2 180)
+		(unit 1)
+		(exclude_from_sim no)
+		(in_bom no)
+		(on_board yes)
+		(dnp no)
+		(property "Reference" "TP6"
+			(at 116.11 82.9 0)
+			(effects
+				(font
+					(size 1.27 1.27)
+				)
+			)
+		)
+		(property "Value" "GND_B"
+			(at 116.11 81 0)
+			(effects
+				(font
+					(size 1.27 1.27)
+				)
+			)
+		)
+		(property "Footprint" "TestPoint:TestPoint_Pad_D1.5mm"
+			(at 120.65 76.2 0)
+			(effects
+				(font
+					(size 1.27 1.27)
+				)
+				(hide yes)
+			)
+		)
+		(property "Datasheet" ""
+			(at 120.65 76.2 0)
+			(effects
+				(font
+					(size 1.27 1.27)
+				)
+				(hide yes)
+			)
+		)
+		(property "Description" "test point"
+			(at 120.65 76.2 0)
+			(effects
+				(font
+					(size 1.27 1.27)
+				)
+				(hide yes)
+			)
+		)
+		(pin "1"
+		)
+		(instances
+			(project "chromatone"
+				(path "/25fa9059-b474-40ad-8d4e-edcbfb8482a5"
+					(reference "TP6")
+					(unit 1)
+				)
