File: boards/chromatone/isolator/isolator.kicad_pcb (KiCad board)
At the start: 2 copper layers, 46 x 30 mm, 23 parts, among them J1 Pi SPI, J2 Strip, U1 ISO7720D

Commit message: chromatone/dac: PCM5102A I2S line-out board (experiment); shared schgen/pcbgen generators
- boardtools/schgen.py and pcbgen.py: the schematic/board generators, extracted
  from the isolator scripts (which now use them and regenerate identically)
- boards/chromatone/dac: schematic + 56x36 mm layout, ERC/DRC clean with parity,
  make jlcpcb runs; README with parts, Pi wiring, config.txt overlay

Co-Authored-By: Claude Fable 5.1 <noreply@anthropic.com>
Other:
- board text added: "chromatone/isolator rev A"
- board text removed: "chromatone rev A"
