File: boards/chromatone/dac/dac.kicad_sch (KiCad schematic)
At the start: 31 parts, among them J1 Pi I2S, J2 Line out, U1 PCM5102A, U2 ME6211C33

Commit message: chromatone/dac: review fixes (audio/XSMT routing off the ground returns, decoupling at pins, full JLCPCB BOM)
Co-Authored-By: Claude Fable 5.1 <noreply@anthropic.com>
Parts:
- C1, C2, C3, C4: LCSC (none) -> C96446; MPN (none) -> CL10A106MA8NRNC; Manufacturer (none) -> Samsung
- C10, C11, C12: LCSC (none) -> C14663; MPN (none) -> CL10B104KB8NNNC; Manufacturer (none) -> Samsung
- C5, C6, C7: LCSC (none) -> C23630; MPN (none) -> CL10A225KO8NNNC; Manufacturer (none) -> Samsung
- C8, C9: LCSC (none) -> C1604; MPN (none) -> 0603B222K500NT; Manufacturer (none) -> Fenghua
- D1: LCSC (none) -> C72043; MPN (none) -> 19-217/GHC-YR1S2/3T; Manufacturer (none) -> Everlight
- R1, R2, R3: LCSC (none) -> C23140; MPN (none) -> 0603WAF330JT5E; Manufacturer (none) -> Uniroyal
- R4, R5: LCSC (none) -> C23179; MPN (none) -> 0603WAF4700T5E; Manufacturer (none) -> Uniroyal
- R6: LCSC (none) -> C25804; MPN (none) -> 0603WAF1002T5E; Manufacturer (none) -> Uniroyal
- R7: LCSC (none) -> C21190; MPN (none) -> 0603WAF1001T5E; Manufacturer (none) -> Uniroyal

Commit message: chromatone/dac: C14663 MPN is Yageo; 4 ms mute-before-power-off
Co-Authored-By: Claude Fable 5.1 <noreply@anthropic.com>
Parts:
- C10, C11, C12: MPN CL10B104KB8NNNC -> CC0603KRX7R9BB104; Manufacturer Samsung -> Yageo
Changed lines of the file:
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@@
 			)
 		)
-		(property "MPN" "CL10B104KB8NNNC"
+		(property "MPN" "CC0603KRX7R9BB104"
 			(at 144.78 73.66 0)
 			(effects
@@
 			)
 		)
-		(property "Manufacturer" "Samsung"
+		(property "Manufacturer" "Yageo"
 			(at 144.78 73.66 0)
 			(effects
@@
 			)
 		)
-		(property "MPN" "CL10B104KB8NNNC"
-			(at 152.4 73.66 0)
-			(effects
-				(font
-					(size 1.27 1.27)
-				)
-				(hide yes)
-			)
-		)
-		(property "Manufacturer" "Samsung"
+		(property "MPN" "CC0603KRX7R9BB104"
+			(at 152.4 73.66 0)
+			(effects
+				(font
+					(size 1.27 1.27)
+				)
+				(hide yes)
+			)
+		)
+		(property "Manufacturer" "Yageo"
 			(at 152.4 73.66 0)
 			(effects
@@
 			)
 		)
-		(property "MPN" "CL10B104KB8NNNC"
+		(property "MPN" "CC0603KRX7R9BB104"
 			(at 160.02 73.66 0)
 			(effects
@@
 			)
 		)
-		(property "Manufacturer" "Samsung"
+		(property "Manufacturer" "Yageo"
 			(at 160.02 73.66 0)
 			(effects
